File: electrical/g3-native/g3-native.kicad_sch (KiCad schematic)
At the start: 44 parts, among them J1 USB_C_Receptacle_USB2.0_16P, J2 Conn_ARM_JTAG_SWD_10, SW1 SW_Push, SW2 SW_Push, U1 STM32H745ZIT6, U2 USBLC6-2SC6, U3 AP2112K-3.3

Commit message: chore: make skeleton for buddies electrical bringup
Parts:
- C1, C2: symbol My Parts:C_10uF_X7R_0805 -> Buddies:C_10uF_X7R_0805
- C10, C11, C12, C13, C14, C15, C16, C18, C20, C21, C22, C23, C24, C29, C3, C4, C5, C6, C7, C8, C9: symbol My Parts:C_100nF_X7R_0402 -> Buddies:C_100nF_X7R_0402
